File: PCB/SDisk2_Simple/SDisk2_Simple.kicad_sch (KiCad schematic)
At the start: 20 parts, among them J2 APPLE II Disk, U1 74HC125, U2 ATmega328P-P, U3 SD_Card_Module, U4 UP, U5 DOWN, U6 ENTER, U7 0.96"OLED_I2C, Y1 27Mhz

Commit message: fixed RESET signal and ERC checks
reset was labeled wrong, it produced a short with VCC
all custom devices' labels were wrong regarding signal direction
Connections:
- net RESET: now reaches R1.1, U2.1 (~{RESET}/PC6)
Other:
- moved on the sheet: R1, R2, R6, U3
